File: AGBM-01 (AA Batteries)/Display.kicad_sch (KiCad schematic)
At the start: 17 parts, among them P2 FFC CONNECTOR

Commit message: Add files via upload
Parts:
- C11: Source (none) -> https://www.digikey.com/short/2ppmm3vt
- C13, C14: Source (none) -> https://www.digikey.com/short/m958w3z3
- C70, C71: Source (none) -> https://www.digikey.com/short/3dr3j004
- P2: Source (none) -> https://www.digikey.com/short/13cnr9vq
- R26: Source (none) -> https://www.digikey.com/short/t0dpzzp1
- R36: Source (none) -> https://www.digikey.com/short/85p4bp5h
- R67, R70, R71: Source (none) -> https://www.digikey.com/short/rpz9t4md
- VR1: Source (none) -> https://www.digikey.com/short/p8zptq5h
- Z57: renamed from C57; value 100p -> 100p or 0 ohm; Source (none) -> https://www.digikey.com/short/h34j0h9q
- Z58: renamed from C58; value 100p -> 100p or 0 ohm; Source (none) -> https://www.digikey.com/short/h34j0h9q
Connections:
- net LA renamed ZA
- net LB renamed ZB
Other:
- note added: "*"
- note added: "*Choose only ONE component! ------------------- Capacitors - touch control Resistors - button trigger"
- note added: "Z70*"
- note added: "Z71*"
- note removed: "Choose only ONE component! ------------------ Capacitor - touch control Resistor - button trigger"
- note removed: "Z70"
- note removed: "Z71"
- company: (none) -> https://github.com/MouseBiteLabs/Game-Boy-Enhance
- moved on the sheet: TP10, TP11, TP31
