File: AGBM-01 (AA Batteries)/CPU.kicad_sch (KiCad schematic)
At the start: 87 parts, among them P1 CART SLOT, P4 AGB-LINK, Q2 NDC7002N, Q7 NDC7002N, Q8 2N7002, SW2 1825027-5, SW3 1825027-5, SW4 SKRRABE010, SW5 SKRRABE010, SW6 SKRRABE010, U1 AGB-CPU, U12 TPS22917DBV, U15 SN74LVC1G332, U16 SN74HC02PWR, U2 AGB-SRAM, X1 4.194304MHz

Commit message: Add files via upload
Parts:
- C15, C16, C17, C34, C39, C43, C5, C52, C53, C6, C7, C8: Source (none) -> https://www.digikey.com/short/m958w3z3
- C18, C19, C20: Source (none) -> https://www.digikey.com/short/h34j0h9q
- C3: Source (none) -> https://www.digikey.com/short/3dr3j004
- C30, C45, C46, C47, C48, C49, C50, C51, C69: Source (none) -> https://www.digikey.com/short/2ppmm3vt
- C4: Source (none) -> https://www.digikey.com/short/q8jbrfqj
- C62, C63, C64, C74, C75, C76, C77, C78: Source (none) -> https://www.digikey.com/short/j50jww8m
- EM1, EM2: Source (none) -> https://www.digikey.com/short/771087dh
- EM3, EM7: Source (none) -> https://www.digikey.com/short/c329ffdd
- P1: Source (none) -> https://tinyurl.com/4uwbr8er
- P4: Source (none) -> https://tinyurl.com/253x94mn
- Q2, Q7: Source (none) -> https://www.digikey.com/short/28n9329f
- Q8: Source (none) -> https://www.digikey.com/short/vbm0z4md
- R1: Source (none) -> https://www.digikey.com/short/pd49zr2b
- R2: Source (none) -> https://www.digikey.com/short/t130htj0
- R29: Source (none) -> https://www.digikey.com/short/1rfwtcff
- R35, R5, R6, R68, R7: Source (none) -> https://www.digikey.com/short/rpz9t4md
- R38, R39: Source (none) -> https://www.digikey.com/short/2trwn31h
- R40, R43, R44: Source (none) -> https://www.digikey.com/short/d1537pn3
- R41: Source (none) -> https://www.digikey.com/short/89v4f1wn
- RA1: Source (none) -> https://www.digikey.com/short/m8cr1b0n
- SW2, SW3: Source (none) -> https://tinyurl.com/36tap2xj
- SW4, SW5, SW6: Source (none) -> https://www.digikey.com/short/2cqndb3b
- U1, U2: Source (none) -> Salvage
- U12: Source (none) -> https://www.digikey.com/short/w4f9v7ht
- U15: Source (none) -> https://www.digikey.com/short/734hmb3p
- U16: Source (none) -> https://www.digikey.com/short/t1r20n2n
- X1: Source (none) -> https://www.digikey.com/short/5t5j99c2
Connections:
- net TP2: now also U16.12; no longer U15.6
- net TP8: now also U15.3; no longer U16.12
- net TP9: now also U15.6; no longer U15.3
- net Display/LA renamed Display/ZA
- net Display/LB renamed Display/ZB
- net LSTSEL renamed LRST
Other:
- sheet Display ports: added ZA, ZB; removed LA, LB
- note added: "L+R+ST"
- note added: "L+R+ST+A"
- note added: "L+R+ST+B"
- note added: "L+R+ST+SEL"
- note added: "L+R+ST+Up"
- note added: "SEL"
- note removed: "L+ST+SEL"
- note removed: "ST+SEL+L+A"
- note removed: "ST+SEL+L+B"
- note removed: "ST+SEL+L+R"
- note removed: "ST+SEL+L+Up"
- company: (none) -> https://github.com/MouseBiteLabs/Game-Boy-Enhance
- moved on the sheet: C39, C78, U15
