File: AGBM-01 (AA Batteries)/AGBM-01_AA_1-2.kicad_pcb (KiCad board)
At the start: 4 copper layers, 131.3 x 72.4 mm, 240 parts, among them P1 CART SLOT, P2 FFC CONNECTOR, P3 SJ-3524-SMT, P4 AGB-LINK, Q1 2N3904, Q10 NDC7002N, Q2 NDC7002N, Q3 2N3906, Q5 NDC7002N, Q6 2N7002, Q7 NDC7002N, Q8 2N7002, Q9 NDC7002N, SW1 CSS-1310B, SW2 1825027-5, SW3 1825027-5, SW4 SKRRABE010, SW5 SKRRABE010, SW6 SKRRABE010, U1 AGB-CPU, U10 TPS3840DL20, U11 TPS22917DBV, U12 TPS22917DBV, U14 MIC1553, U15 SN74LVC1G332, U16 SN74HC02PWR, U17 TPS3840DL20, U18 TPS22917DBV, U2 AGB-SRAM, U3 TPS3840DL20, U4 NCV8164ASN250T1G, U5 LTC3527, U6 LM4853, U7 TLV9364, U8 NCV8164ASN250T1G, U9 SN74LVC2G34DBVR, X1 4.194304MHz

Commit message: Add files via upload
Parts:
- TP22: value BATT -> VAUD
