File: AGBM-01 (AA Batteries)/AGBM-01_AA_1-2.kicad_sch (KiCad schematic)
At the start: 81 parts, among them Q1 2N3904, Q10 NDC7002N, Q3 2N3906, Q5 NDC7002N, Q9 NDC7002N, SW1 CSS-1310B, U10 TPS3840DL20, U11 TPS22917DBV, U14 MIC1553, U17 TPS3840DL20, U18 TPS22917DBV, U3 TPS3840DL20, U4 NCV8164ASN250T1G, U5 LTC3527, U8 NCV8164ASN250T1G

Commit message: Add files via upload
Parts:
- R3: value 1k -> 5.1k
- R4: value 10k -> 33k
Other:
- note added: "Cutoff: 2.3V"
- note removed: "Cutoff: 2.2V"
Changed lines of the file:
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@@
 		)
 	)
-	(text "Cutoff: 2.2V"
+	(text "Cutoff: 2.3V"
 		(exclude_from_sim no)
 		(at 205.232 44.45 0)
@@
 			)
 		)
-		(property "Value" "10k"
+		(property "Value" "33k"
 			(at 206.756 53.086 0)
 			(effects
@@
 			)
 		)
-		(property "Value" "1k"
+		(property "Value" "5.1k"
 			(at 196.596 40.386 0)
 			(effects
@@
 		)
 		(instances
-			(project "AGBM_AA_1-2"
+			(project "AGBM-01_AA_1-2"
 				(path "/cfd0659f-d3b3-4ed9-9d9b-b9f1ae0cdd25"
 					(page "2")

Commit message: Add files via upload
Parts:
- R3: Source https://www.digikey.com/short/nwddb5fm -> https://www.digikey.com/short/qqj3r2v5
- R4: Source https://www.digikey.com/short/t130htj0 -> https://www.digikey.com/short/t0dpzzp1
- R64: value 100k -> 200k; Source https://www.digikey.com/short/rpz9t4md -> https://www.digikey.com/short/3391593q
Changed lines of the file:
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@@
 			)
 		)
-		(property "Value" "100k"
+		(property "Value" "200k"
 			(at 271.272 88.646 0)
 			(effects
@@
 			)
 		)
-		(property "Source" "https://www.digikey.com/short/rpz9t4md"
+		(property "Source" "https://www.digikey.com/short/3391593q"
 			(at 273.05 87.63 0)
 			(effects
@@
 			)
 		)
-		(property "Source" "https://www.digikey.com/short/t130htj0"
+		(property "Source" "https://www.digikey.com/short/t0dpzzp1"
 			(at 208.28 52.07 0)
 			(effects
@@
 			)
 		)
-		(property "Source" "https://www.digikey.com/short/nwddb5fm"
+		(property "Source" "https://www.digikey.com/short/qqj3r2v5"
 			(at 198.12 39.37 0)
 			(effects
