File: AGBM-11 (Lithium-ion)/Audio.kicad_sch (KiCad schematic)
At the start: 50 parts, among them P3 SJ-3524-SMT, Q6 2N7002, U6 LM4853, U7 TLV9364, U9 SN74LVC2G34DBVR

Commit message: Add files via upload
Parts:
- C24, C32: Source https://www.digikey.com/short/377h8558 -> (none)
- C25, C29, C36, C38, C54, C55, C56, C9: Source https://www.digikey.com/short/2ppmm3vt -> (none)
- C26, C31: Source https://www.digikey.com/short/jm5qjr7w -> (none)
- C27, C33: Source https://www.digikey.com/short/5ptw22qq -> (none)
- C28, C35: Source https://www.digikey.com/short/3p3jj3wt -> (none)
- CP1, CP2, CP3: Source https://www.digikey.com/short/332b01qh -> (none)
- P3: footprint Bucketmouse:CUI_SJ-3524-SMT -> Bucketmouse:SJ3-35083B-TR_AND_SJ-3524-SMT; SnapEDA_Link (none) -> https://www.snapeda.com/parts/SJ-3524-SMT-TR/Same+Sky/view-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; Source https://www.digikey.com/short/r4b2bq43 -> (none)
- Q6: Source https://www.digikey.com/short/vbm0z4md -> (none)
- R14, R30, R31, R37, R45, R46, R49, R50: Source https://www.digikey.com/short/rpz9t4md -> (none)
- R19, R20: Source https://www.digikey.com/short/nwddb5fm -> (none)
- R34, R53: Source https://www.digikey.com/short/qqj3r2v5 -> (none)
- R42, R51: Source https://www.digikey.com/short/vn4221jt -> (none)
- R47, R52, R56, R57: Source https://www.digikey.com/short/38d0p2b4 -> (none)
- R48, R54: Source https://www.digikey.com/short/1rfwtcff -> (none)
- SP1: Source https://tinyurl.com/yxxmec4w -> (none)
- U6: Source https://www.digikey.com/short/r3rqdzt8 -> (none)
- U7: Source https://www.digikey.com/short/jhr04t1t -> (none)
- U9: Source https://www.digikey.com/short/tzhnmjv0 -> (none)
- VR2: Source https://www.digikey.com/short/zh4rmq4h -> (none)
Other:
- company: https://github.com/MouseBiteLabs/Game-Boy-Enhance -> https://github.com/MouseBiteLabs/Game-Boy-Enhance/
- title: Game Boy Enhance (AGBM-01) -> Game Boy Enhance (AGBM-11)
