File: AGBM-11 (Lithium-ion)/CPU.kicad_sch (KiCad schematic)
At the start: 87 parts, among them P1 CART SLOT, P4 AGB-LINK, Q2 NDC7002N, Q7 NDC7002N, Q8 2N7002, SW2 1825027-5, SW3 1825027-5, SW4 SKRRABE010, SW5 SKRRABE010, SW6 SKRRABE010, U1 AGB-CPU, U12 TPS22917DBV, U15 SN74LVC1G332, U16 SN74HC02PWR, U2 AGB-SRAM, X1 4.194304MHz

Commit message: Add files via upload
Parts:
- removed TP25: SCK, Bucketmouse:TestPoint_Pad_D1.0mm, symbol OpenGBA:TestPoint
- added TP35: SCK, Bucketmouse:TestPoint_Pad_D1.0mm, symbol OpenGBA:TestPoint
- C15, C16, C17, C34, C39, C43, C5, C52, C53, C6, C7, C8: Source https://www.digikey.com/short/m958w3z3 -> (none)
- C18, C19, C20: Source https://www.digikey.com/short/h34j0h9q -> (none)
- C3: Source https://www.digikey.com/short/3dr3j004 -> (none)
- C30, C45, C46, C47, C48, C49, C50, C51, C69: Source https://www.digikey.com/short/2ppmm3vt -> (none)
- C4: Source https://www.digikey.com/short/q8jbrfqj -> (none)
- C62, C63, C64, C74, C75, C76, C77, C78: Source https://www.digikey.com/short/j50jww8m -> (none)
- EM1, EM2: Source https://www.digikey.com/short/771087dh -> (none)
- EM3, EM7: Source https://www.digikey.com/short/c329ffdd -> (none)
- P1: Source https://tinyurl.com/4uwbr8er -> (none)
- P4: Source https://tinyurl.com/253x94mn -> (none)
- Q2, Q7: Source https://www.digikey.com/short/28n9329f -> (none)
- Q8: Source https://www.digikey.com/short/vbm0z4md -> (none)
- R1: Source https://www.digikey.com/short/pd49zr2b -> (none)
- R2: Source https://www.digikey.com/short/t130htj0 -> (none)
- R29: Source https://www.digikey.com/short/1rfwtcff -> (none)
- R35, R5, R6, R68, R7: Source https://www.digikey.com/short/rpz9t4md -> (none)
- R38, R39: Source https://www.digikey.com/short/2trwn31h -> (none)
- R40, R43, R44: Source https://www.digikey.com/short/d1537pn3 -> (none)
- R41: Source https://www.digikey.com/short/89v4f1wn -> (none)
- RA1: Source https://www.digikey.com/short/m8cr1b0n -> (none)
- SW2, SW3: value 1825027-5 -> SW_Push; Source https://tinyurl.com/36tap2xj -> (none)
- SW4, SW5, SW6: value SKRRABE010 -> ~; Source https://www.digikey.com/short/2cqndb3b -> (none)
- U1, U2: Source Salvage -> (none)
- U12: Source https://www.digikey.com/short/w4f9v7ht -> (none)
- U15: Source https://www.digikey.com/short/734hmb3p -> (none)
- U16: Source https://www.digikey.com/short/t1r20n2n -> (none)
- X1: Source https://www.digikey.com/short/5t5j99c2 -> (none)
Connections:
- net at EM2.2, RA1.8 (R1.2): now also TP35.1
Other:
- company: https://github.com/MouseBiteLabs/Game-Boy-Enhance -> https://github.com/MouseBiteLabs/Game-Boy-Enhance/
- title: Game Boy Enhance (AGBM-01) -> Game Boy Enhance (AGBM-11)
