File: AGBM-11 (Lithium-ion)/AGBM-11_LiPo_1-2.kicad_pcb (KiCad board)
At the start: 4 copper layers, 131.3 x 73.9 mm, 258 parts, among them J1 JST-SH, J2 Conn_01x02_Socket, P1 CART SLOT, P2 FFC CONNECTOR, P3 SJ-3524-SMT, P4 AGB-LINK, P5 USB-C-6P, Q1 2N3904, Q10 NDC7002N, Q2 NDC7002N, Q3 2N3906, Q4 NTGD3148, Q5 NDC7002N, Q6 2N7002, Q7 NDC7002N, Q8 2N7002, Q9 NDC7002N, SW1 CSS-1X10B, SW2 SW_Push, SW3 SW_Push, U1 AGB-CPU, U10 TPS3840DL30, U11 TPS22917DBV, U12 TPS22917DBV, U13 S-82M1A, U14 MIC1553, U15 SN74LVC1G332, U16 SN74HC02PWR, U17 TPS3840DL30, U19 MCP73871-2CAI/ML, U2 AGB-SRAM, U3 TPS3840DL30, U4 NCV8164ASN250T1G, U5 LTC3527, U6 LM4853, U7 TLV9364, U8 NCV8164ASN250T1G, U9 SN74LVC2G34DBVR, X1 4.194304MHz

Commit message: Add files via upload
Parts:
- TP22: value BATT -> VAUD
Changed lines of the file:
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@@
 			)
 		)
-		(property "Value" "BATT"
-			(at 0 -2.6 90)
+		(property "Value" "VAUD"
+			(at 0 -2.95 90)
 			(unlocked yes)
 			(layer "F.SilkS")
@@
 		(tags "resistor")
 		(property "Reference" "R33"
-			(at -1.9 -2.4 0)
+			(at -2.2 -2.4 0)
 			(unlocked yes)
 			(layer "B.SilkS")
@@
 			)
 		)
+		(model "${KICAD9_3DMODEL_DIR}/Connector_JST.3dshapes/SM02B-SRSS-TB-LF--SN---3DModel-STEP-56544.STEP"
+			(offset
+				(xyz 0 1 0)
+			)
+			(scale
+				(xyz 1 1 1)
+			)
+			(rotate
+				(xyz -90 -0 -0)
+			)
+		)
 	)
 	(footprint "Bucketmouse:C_0603_1608Metric_Boxed_2"
@@
 			)
 		)
+		(model "${KICAD9_3DMODEL_DIR}/Package_DFN_QFN.3dshapes/QFN-20-1EP_4x4mm_P0.5mm_EP2.5x2.5mm.step"
+			(offset
+				(xyz 0 0 0)
+			)
+			(scale
+				(xyz 1 1 1)
+			)
+			(rotate
+				(xyz 0 0 0)
+			)
+		)
 	)
 	(footprint "Bucketmouse:C_0603_1608Metric_Boxed_2"
@@
 		)
 		(embedded_fonts no)
+		(model "${KICAD9_3DMODEL_DIR}/Button_Switch_SMD.3dshapes/CSS-1310TB.step"
+			(offset
+				(xyz 0.6 -1.2 1)
+			)
+			(scale
+				(xyz 1 1 1)
+			)
+			(rotate
+				(xyz -90 -0 -0)
+			)
+		)
 	)
 	(footprint "Bucketmouse:C_0603_1608Metric_Boxed_2"
@@
 		)
 		(embedded_fonts no)
-		(model "${KICAD9_3DMODEL_DIR}/Battery.3dshapes/Battery_CR1225.step"
+		(model "${KICAD9_3DMODEL_DIR}/Potentiometer_SMD.3dshapes/Unnamed-SOLID.step"
 			(offset
 				(xyz 0 0 0)
 			)
 			(scale
-				(xyz 1.1 1.1 1)
+				(xyz 1 1 1)
 			)
 			(rotate
@@
 		)
 		(embedded_fonts no)
+		(model "${KICAD9_3DMODEL_DIR}/Connector_Audio.3dshapes/Same_Sky_SJ3-35083B-TR.step"
+			(offset
+				(xyz 11 0 2.5)
+			)
+			(scale
+				(xyz 1 1 1)
+			)
+			(rotate
+				(xyz 90 180 -90)
+			)
+		)
 	)
 	(footprint "Bucketmouse:R_0603_1608Metric_Boxed"
@@
 	)
 	(gr_circle
-		(center 125.7 -20)
-		(end 125.7 -20.125)
+		(center 125.1 -19.4)
+		(end 125.1 -19.525)
 		(stroke
 			(width 0.2)
