File: AGBM-11 (Lithium-ion)/AGBM-11_LiPo_1-2.kicad_sch (KiCad schematic)
At the start: 98 parts, among them J1 JST-SH, J2 Conn_01x02_Socket, P5 USB-C-6P, Q1 2N3904, Q10 NDC7002N, Q3 2N3906, Q4 NTGD3148, Q5 NDC7002N, Q9 NDC7002N, SW1 CSS-1X10B, U10 TPS3840DL30, U11 TPS22917DBV, U13 S-82M1A, U14 MIC1553, U17 TPS3840DL30, U19 MCP73871-2CAI/ML, U3 TPS3840DL30, U4 NCV8164ASN250T1G, U5 LTC3527, U8 NCV8164ASN250T1G

Commit message: Add files via upload
Parts:
- R3: value 1k -> 3.3k
- R63: value 30k -> 15k
Other:
- note added: "Cutoff: 3.2V"
- note added: "Cutoff: 3.5V"
- note removed: "Cutoff: 3.15V"
- note removed: "Cutoff: 3.1V"
Changed lines of the file:
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@@
 		)
 	)
-	(text "Cutoff: 3.1V"
+	(text "Cutoff: 3.2V"
 		(exclude_from_sim no)
 		(at 205.232 91.44 0)
@@
 		)
 	)
-	(text "Cutoff: 3.15V"
+	(text "Cutoff: 3.5V"
 		(exclude_from_sim no)
 		(at 205.232 49.53 0)
@@
 			)
 		)
-		(property "Value" "30k"
+		(property "Value" "15k"
 			(at 206.756 98.806 0)
 			(effects
@@
 			)
 		)
-		(property "Value" "1k"
+		(property "Value" "3.3k"
 			(at 196.596 45.466 0)
 			(effects
